Commit message: lets see what happens

File: bluerov_uuv/models/rexrov/urdf/rexrov_base.xacro (robot description, xacro)
@@ -86,5 +86,5 @@
         <origin xyz="0 0 0" rpy="0 0 0"/>
         <geometry>
-          <mesh filename="${visual_mesh_file}" scale="0.001 0.001 0.001"/>
+          <mesh filename="${visual_mesh_file}" scale="0.005 0.005 0.005"/>
         </geometry>
       </visual>
