Commit message: Hydrodynamics still messed up

File: enigma_description/urdf/base.xacro (robot description, xacro)
@@ -43,5 +43,5 @@
           <origin xyz="0 0 0" rpy="0 0 0"/>
           <geometry>
-            <mesh filename="${visual_mesh_file}" scale="0.01 0.01 0.01" />
+            <mesh filename="${visual_mesh_file}" scale="0.003 0.003 0.003" />
           </geometry>
         </visual>

Commit message: chalo bhaiya

File: enigma_description/urdf/base.xacro (robot description, xacro)
@@ -21,5 +21,5 @@
     Open the meshes for the RexROV vehicle in Blender to see an example on the mesh placement.
   -->
-  <xacro:property name="visual_mesh_file" value="file://$(find enigma_description)/meshes/bluerov.dae"/>
+  <xacro:property name="visual_mesh_file" value="file://$(find enigma_description)/meshes/fixed_rov.dae"/>
   <!-- <xacro:property name="visual_mesh_file" value="file://$(find enigma_description)/meshes/rex.dae"/> -->
   <!-- Collision geometry mesh, usually in STL format (it is recommended to keep

Commit message: Bluerov finally working

File: enigma_description/urdf/base.xacro (robot description, xacro)
@@ -43,5 +43,5 @@
           <origin xyz="0 0 0" rpy="0 0 0"/>
           <geometry>
-            <mesh filename="${visual_mesh_file}" scale="0.003 0.003 0.003" />
+            <mesh filename="${visual_mesh_file}" scale="1 1 1" />
           </geometry>
         </visual>
