Commit message: I am trying

File: enigma_description/urdf/actuators.xacro (robot description, xacro)
@@ -9,14 +9,23 @@
     -->
     <xacro:thruster_macro robot_namespace="${namespace}" thruster_id="0">
-        <origin xyz="0 0 0" rpy="0 0 ${pi}" />
+        <origin xyz="0.0 0.115 0.0" rpy="-0.0 -1.57079632679 0.0"/>
     </xacro:thruster_macro>
     <xacro:thruster_macro robot_namespace="${namespace}" thruster_id="1">
-        <origin xyz="0 0 0" rpy="0 0 ${pi}" />
+        <origin xyz="0.0 -0.115 0.0" rpy="-0.0 -1.57079632679 0.0"/>
     </xacro:thruster_macro>
     <xacro:thruster_macro robot_namespace="${namespace}" thruster_id="2">
-    <origin xyz="0 0 0" rpy="0 -${0.5*pi} 0" />
+      <origin xyz="0.18 0.1092 0.0" rpy="0.0 -0.0 0.0"/>
+    </xacro:thruster_macro>
+    <xacro:thruster_macro robot_namespace="${namespace}" thruster_id="3">
+      <origin xyz="0.18 -0.1092 0.0" rpy="0.0 -0.0 0.0"/>
+    </xacro:thruster_macro>
+    <xacro:thruster_macro robot_namespace="${namespace}" thruster_id="4">
+      <origin  xyz="-0.17 0.0 0.0" rpy="0.0 -0.0 0.0"/>
+    </xacro:thruster_macro>
+    <xacro:thruster_macro robot_namespace="${namespace}" thruster_id="5">
+      <origin xyz="0.0 0.0 0.105" rpy="1.57079632679 -0.0 0.0"/>
     </xacro:thruster_macro>
     <!-- Instantiate fins, if necessary -->
-    <xacro:fin_macro namespace="${namespace}" fin_id="0">
+    <!-- <xacro:fin_macro namespace="${namespace}" fin_id="0">
       <origin xyz="0 0 0" rpy="0 0 0" />
     </xacro:fin_macro>
@@ -29,4 +38,4 @@
     <xacro:fin_macro namespace="${namespace}" fin_id="3">
       <origin xyz="0 0 0" rpy="0 0 0" />
-    </xacro:fin_macro>
+    </xacro:fin_macro> -->
 </robot>

File: enigma_description/urdf/base.xacro (robot description, xacro)
@@ -6,5 +6,5 @@
   <xacro:include filename="$(find uuv_sensor_plugins_ros)/urdf/sensor_snippets.xacro"/>
   <!-- Loading vehicle's specific macros -->
-  <!-- <xacro:include filename="$(find enigma_description)/urdf/snippets.xacro"/> -->
+  <xacro:include filename="$(find enigma_description)/urdf/snippets.xacro"/>
   <!--
     Vehicle's parameters (remember to enter the model parameters below)

File: enigma_description/urdf/snippets.xacro (robot description, xacro)
@@ -7,10 +7,10 @@
   over propeller's frame X-axis in DAE (Collada) or STL format.
   -->
-  <xacro:property name="prop_mesh_file" value="file://$(find enigma_description)/meshes/propeller.dae"/>
+  <!-- <xacro:property name="prop_mesh_file" value="file://$(find enigma_description)/meshes/propeller.dae"/> -->
   <!--
     Thruster macro with integration of joint and link. The thrusters should
     be initialized in the actuators.xacro file.
   -->
-  <xacro:macro name="thruster_macro" params="robot_namespace thruster_id *origin">
+  <!-- <xacro:macro name="thruster_macro" params="robot_namespace thruster_id *origin"> -->
     <!--
     Dummy link as place holder for the thruster frame,
@@ -18,5 +18,5 @@
     of the vehicle and may cause internal collisions if set otherwise
     -->
-    <link name="${robot_namespace}/thruster_${thruster_id}">
+    <!-- <link name="${robot_namespace}/thruster_${thruster_id}">
       <visual>
         <geometry>
@@ -31,127 +31,26 @@
                izz="0.000000017" />
       </inertial>
-    </link>
+    </link> -->
     <!-- Joint between thruster link and vehicle base link -->
-    <joint name="${robot_namespace}/thruster_${thruster_id}_joint" type="continuous">
+    <!-- <joint name="${robot_namespace}/thruster_${thruster_id}_joint" type="continuous">
       <xacro:insert_block name="origin" />
       <axis xyz="1 0 0" />
       <parent link="${robot_namespace}/base_link" />
       <child link="${robot_namespace}/thruster_${thruster_id}" />
-    </joint>
-    <gazebo>
-      <!-- Thruster ROS plugin -->
-      <plugin name="${robot_namespace}_${thruster_id}_thruster_model" filename="libthruster_ros_plugin.so">
-        <!-- Name of the thruster link -->
-        <linkName>${robot_namespace}/thruster_${thruster_id}</linkName>
-        <!-- Name of the joint between thruster and vehicle base link -->
-        <jointName>${robot_namespace}/thruster_${thruster_id}_joint</jointName>
-        <!-- Make the thruster aware of its id -->
-        <thrusterId>${thruster_id}</thrusterId>
-        <!-- Gain of the input command signal -->
-        <gain>1</gain>
-        <!-- Maximum allowed input value for the input signal for thruster unit -->
-        <clampMax>0</clampMax>
-        <!-- Minimum allowed value for the input signal for thruster unit -->
-        <clampMin>0</clampMin>
-        <!-- Minimum and maximum thrust force output allowed -->
-        <thrustMin>0</thrustMin>
-        <thrustMax>0</thrustMax>
-        <!--
-        Value from 0 to 1 to set the efficiency of the output thrust force
-        Default value is 1.0
-        -->
-        <thrust_efficiency>1</thrust_efficiency>
-        <!--
-        Value from 0 to 1 to set the efficiency of the propeller as a factor
-        to be multiplied to the current value of the state variable at each
-        iteration.
-        Default value is 1.0
-        -->
-        <propeller_efficiency>1</propeller_efficiency>
-        <!--
-        ----------------------------------------------------
-        ----------------------------------------------------
-        Choose one of the propeller dynamics models below for your implementation
-        This will describe the dynamic model for the state variable of your thruster unit,
-        which can be, e.g., the angular velocity of the propeller.
-        ----------------------------------------------------
-        ---------------------------------------------------->
-        <!-- 1) Simple zero-order model -->
-        <dynamics>
-          <type>ZeroOrder</type>
-        </dynamics>
-        <!-- 2) First order model -->
+    </joint> -->
+  <!-- <xacro:property name="prop_mesh_file" value="file://$(find uuv_descriptions)/models/rexrov/mesh/prop.dae"/> -->
+  <!-- Thruster joint and link snippet -->
+    <!-- <gazebo>
+      <plugin name="${namespace}_${thruster_id}_thruster_model" filename="libthruster_ros_plugin.so">
+        <linkName>${namespace}/thruster_${thruster_id}</linkName>
+        <jointName>${namespace}/thruster_${thruster_id}_joint</jointName>
+        <thrusterID>${thruster_id}</thrusterID>
         <dynamics>
           <type>FirstOrder</type>
-          <timeConstant>0.0</timeConstant>
+          <timeConstant>0.05</timeConstant>urdf
         </dynamics>
-        <!-- 3) Yoerger's nonlinear dynamic model
-        For information on the model description:
-        [1] D. R. Yoerger, J. G. Cooke, and J.-J. E. Slotine, “The influence of
-            thruster dynamics on underwater vehicle behavior and their incorporation
-            into control system design,” IEEE Journal of Oceanic Engineering, vol. 15,
-            no. 3, pp. 167–178, Jul. 1990.
-        -->
-        <dynamics>
-          <type>Yoerger</type>
-          <alpha>0.0</alpha>
-          <beta>0.0</beta>
-        </dynamics>
-        <!-- 4) Bessa's nonlinear dynamic model
-        For information on the model description:
-        [2] Bessa, Wallace Moreira, Max Suell Dutra, and Edwin Kreuzer. "Thruster
-            dynamics compensation for the positioning of underwater robotic vehicles
-            through a fuzzy sliding mode based approach." ABCM Symposium Series in
-            Mechatronics. Vol. 2. 2006.
-        -->
-        <dynamics>
-          <type>Bessa</type>
-          <Jmsp>0.0</Jmsp>
-          <Kv1>0.0</Kv1>
-          <Kv2>0.0</Kv2>
-          <Kt>0.0</Kt>
-          <Rm>0.0</Rm>
-        </dynamics>
-        <!--
-        ----------------------------------------------------
-        ----------------------------------------------------
-        Choose one of the model for the steady-state curve describing the
-        relationship between the state variable and the output thrust force
-        ----------------------------------------------------
-        ---------------------------------------------------->
-        <!-- 1) Basic curve
-        Input: x
-        Output: thrust
-        Function: thrust = rotorConstant * x * abs(x)
-        -->
         <conversion>
           <type>Basic</type>
-          <rotorConstant>0.0</rotorConstant>
-        </conversion>
-        <!-- 2) Dead-zone nonlinearity described in Bessa, 2006
-        Input: x
-        Output: thrust
-        Function:
-        thrust = rotorConstantL * (x * abs(x) - deltaL), if x * abs(x) <= deltaL
-        thrust = 0, if deltaL < x * abs(x) < deltaR
-        thrust = rotorConstantR * (x * abs(x) - deltaR), if x * abs(x) >= deltaL
-        -->
-        <conversion>
-          <type>Bessa</type>
-          <rotorConstantL>0.0</rotorConstantL>
-          <rotorConstantR>0.0</rotorConstantR>
-          <deltaL>0.0</deltaL>
-          <deltaR>0.0</deltaR>
-        </conversion>
-        <!-- 3) Linear interpolation
-        If you have access to the thruster's data sheet, for example,
-        you can enter samples of the curve's input and output values
-        and the thruster output will be found through linear interpolation
-        of the given samples.
-        -->
-        <conversion>
-          <type>LinearInterp</type>
-          <inputValues>0 1 2 3</inputValues>
-          <outputValues>0 1 2 3</outputValues>
+          <rotorConstant>0.00031</rotorConstant>
         </conversion>
       </plugin>
@@ -160,4 +59,4 @@
       <selfCollide>false</selfCollide>
     </gazebo>
-  </xacro:macro>
+  </xacro:macro> -->
 </robot>

Commit message: haha

File: enigma_description/urdf/actuators.xacro (robot description, xacro)
@@ -8,32 +8,30 @@
           aware that Gazebo does not use the SNAME convention per default.
     -->
-<!--    <xacro:macro name="thruster_macro"
+   <xacro:macro name="thruster_macro"
     params="namespace thruster_id *origin">
-    <xacro:thruster_module_first_order_basic_fcn_macro
+    <xacro:thruster_module_first_order_basic_fcn_macro_nomesh
       namespace="${namespace}"
       thruster_id="${thruster_id}"
       dyn_time_constant="0.05"
-      mesh_filename=""
       rotor_constant="0.00031">
-      <xacro:insert_block name="origin"/>
-    </xacro:thruster_module_first_order_basic_fcn_macro>
+      <!-- <xacro:insert_block name="origin"/> -->
+    </xacro:thruster_module_first_order_basic_fcn_macro_nomesh>
   </xacro:macro>
- -->
-    <xacro:thruster_macro robot_namespace="${namespace}" thruster_id="0">
+    <xacro:thruster_macro namespace="${namespace}" thruster_id="0">
         <origin xyz="0.0 0.115 0.0" rpy="-0.0 -1.57079632679 0.0"/>
     </xacro:thruster_macro>
-    <xacro:thruster_macro robot_namespace="${namespace}" thruster_id="1">
+    <xacro:thruster_macro namespace="${namespace}" thruster_id="1">
         <origin xyz="0.0 -0.115 0.0" rpy="-0.0 -1.57079632679 0.0"/>
     </xacro:thruster_macro>
-    <xacro:thruster_macro robot_namespace="${namespace}" thruster_id="2">
-      <origin xyz="0.18 0.1092 0.0" rpy="0.0 -0.0 0.0"/>
+    <xacro:thruster_macro namespace="${namespace}" thruster_id="2">
+  gin xyz="0.18 0.1092 0.0" rpy="0.0 -0.0 0.0"/>
     </xacro:thruster_macro>
-    <xacro:thruster_macro robot_namespace="${namespace}" thruster_id="3">
+    <xacro:thruster_macro namespace="${namespace}" thruster_id="3">
       <origin xyz="0.18 -0.1092 0.0" rpy="0.0 -0.0 0.0"/>
     </xacro:thruster_macro>
-    <xacro:thruster_macro robot_namespace="${namespace}" thruster_id="4">
+    <xacro:thruster_macro namespace="${namespace}" thruster_id="4">
       <origin  xyz="-0.17 0.0 0.0" rpy="0.0 -0.0 0.0"/>
     </xacro:thruster_macro>
-    <xacro:thruster_macro robot_namespace="${namespace}" thruster_id="5">
+    <xacro:thruster_macro namespace="${namespace}" thruster_id="5">
       <origin xyz="0.0 0.0 0.105" rpy="1.57079632679 -0.0 0.0"/>
     </xacro:thruster_macro>

File: enigma_description/urdf/base.xacro (robot description, xacro)
@@ -6,6 +6,6 @@
   <xacro:include filename="$(find uuv_sensor_plugins_ros)/urdf/sensor_snippets.xacro"/>
   <!-- Loading vehicle's specific macros -->
-  <xacro:include filename="$(find enigma_description)/urdf/snippets.xacro"/>
-  <!-- <xacro:include filename="$(find uuv_gazebo_ros_plugins)/urdf/snippets.xacro"/> -->
+  <!-- <xacro:include filename="$(find enigma_description)/urdf/snippets.xacro"/> -->
+  <xacro:include filename="$(find uuv_gazebo_ros_plugins)/urdf/snippets.xacro"/>
   <!--
     Vehicle's parameters (remember to enter the model parameters below)
