Commit message: updated bluerov launch

File: bluerov_uuv/models/bluerov/urdf/bluerov_base.xacro (robot description, xacro)
@@ -10,16 +10,18 @@
     Vehicle's parameters
   -->
-  <xacro:property name="mass" value="0"/>
-  <xacro:property name="volume" value="0"/>
+  <!-- Mass in Kg, and length measurements in m-->
+  <xacro:property name="mass" value="12"/>
+  <xacro:property name="volume" value="0.05"/>
   <!-- Center of gravity -->
-  <xacro:property name="cog" value="0 0 0"/>
+  <xacro:property name="cog" value="0.24 0.165 0.22"/>
   <!-- Center of buoyancy -->
-  <xacro:property name="cob" value="0 0 0"/>
+  <xacro:property name="cob" value="0.24 0.165 0.22"/>
   <!-- Fluid density -->
   <xacro:property name="rho" value="1028"/>
+  <xacro:property name="PI" value="3.1415926535897931"/>
   <!-- Describing the dimensions of the vehicle's bounding box -->
-  <xacro:property name="length" value="0"/>
-  <xacro:property name="width"  value="0"/>
-  <xacro:property name="height" value="0"/>
+  <xacro:property name="length" value="0.48"/>
+  <xacro:property name="width"  value="0.33"/>
+  <xacro:property name="height" value="0.38"/>
   <!-- Visual mesh file for the vehicle, usually in DAE (Collada) format -->
   <xacro:property name="visual_mesh_file" value="file://$(find bluerov_uuv)/models/bluerov/mesh/bluerov.dae"/>
@@ -27,5 +29,5 @@
   this geometry as simple as possible to improve the performance the physics engine
   regarding the computation of collision forces) -->
-  <xacro:property name="collision_mesh_file" value="file://$(find bluerov_uuv)/models/bluerov/mesh/vehicle.stl"/>
+  <xacro:property name="collision_mesh_file" value="file://$(find bluerov_uuv)/models/bluerov/mesh/collision.blend"/>
   <!-- Vehicle macro -->
   <xacro:macro name="bluerov_base" params="namespace debug">
@@ -35,12 +37,12 @@
         <mass value="${mass}" />
         <origin xyz="${cog}" rpy="0 0 0"/>
-        <inertia ixx="0" ixy="0" ixz="0"
-                 iyy="0" iyz="0"
-                 izz="0" />
+        <inertia ixx="5" ixy="0.0" ixz="0.0"
+                 iyy="5" iyz="5"
+                 izz="5" />
       </inertial>
       <visual>
-        <origin xyz="0 0 0" rpy="0 0 0"/>
+        <origin xyz="-0.241 0.165 0.17" rpy="${-PI/2} 0 -${PI/2}"/>
         <geometry>
-          <mesh filename="${visual_mesh_file}" scale="1 1 1" />
+          <mesh filename="${visual_mesh_file}" scale="0.001 0.001 0.001" />
         </geometry>
       </visual>
@@ -54,4 +56,10 @@
   <gazebo reference="${namespace}/base_link">
     <selfCollide>false</selfCollide>
+  </gazebo>
+  <gazebo>
+      <!-- optional: plugin to test compare Gazebo's returned accelerations -->
+    <plugin name="${namespace}_test_plugin" filename="libaccelerations_test_plugin.so">
+      <link_name>${namespace}/base_link</link_name>
+    </plugin>
   </gazebo>
   <!-- Dummy link for the frame in SNAME standard, Gazebo does not offer
@@ -92,48 +100,24 @@
           <!-- Center of buoyancy -->
           <center_of_buoyancy>${cob}</center_of_buoyancy>
-          <!--
-          ----------------------------------------------------
-          ----------------------------------------------------
-          Choose one of the hydrodynamic models below, all are based on
-          Fossen's equation of motion for underwater vehicles
-          Reference:
-          Fossen, Thor I. Handbook of marine craft hydrodynamics and motion
-          control. John Wiley & Sons, 2011.
-          ----------------------------------------------------
-          ---------------------------------------------------->
           <!-- Fossen's equation of motion -->
           <hydrodynamic_model>
-            <type>fossen</type>
-            <added_mass>
-              0 0 0 0 0 0
-              0 0 0 0 0 0
-              0 0 0 0 0 0
-              0 0 0 0 0 0
-              0 0 0 0 0 0
-              0 0 0 0 0 0
-            </added_mass>
-            <!--
-            The linear damping coefficients can be provided as a diagonal (6 elements)
-            or a full matrix (36 coefficients), like the added-mass coefficients above
-            -->
-            <linear_damping>
-              0 0 0 0 0 0
-            </linear_damping>
-            <!--
-            The linear damping coefficients proportional to the forward speed
-            can be provided as a diagonal (6 elements) or a full matrix (36 coefficients),
-            like the added-mass coefficients above.
-            This matrix is mostly useful for slender bodies (e.g. AUVs with torpedo shape)
-            -->
-            <linear_damping_forward_speed>
-              0 0 0 0 0 0
-            </linear_damping_forward_speed>
-            <!--
-            The quadratic damping coefficients can be provided as a diagonal (6 elements)
-            or a full matrix (36 coefficients), like the added-mass coefficients above
-            -->
-            <quadratic_damping>
-              0 0 0 0 0 0
-            </quadratic_damping>
+                 <type>fossen</type>
+                 <!-- Added mass: see p.28 in Berg2012 -->
+                 <added_mass>
+                      779.79 -6.8773 -103.32  8.5426 -165.54 -7.8033
+                     -6.8773    1222   51.29  409.44 -5.8488  62.726
+                     -103.32   51.29  3659.9  6.1112 -386.42  10.774
+                      8.5426  409.44  6.1112   534.9 -10.027  21.019
+                     -165.54 -5.8488 -386.42 -10.027  842.69 -1.1162
+                     -7.8033  62.726  10.775  21.019 -1.1162  224.32
+                 </added_mass>
+                 <!-- Linear damping: see p.31 in Berg2012 -->
+                 <linear_damping>
+                     -74.82 -69.48 -728.4 -268.8 -309.77 -105
+                 </linear_damping>
+                 <!-- Non-linear damping: see p.30 in Berg2012 -->
+                 <quadratic_damping>
+                     -748.22 -992.53 -1821.01 -672 -774.44 -523.27
+                 </quadratic_damping>
           </hydrodynamic_model>
         </link>

File: bluerov_uuv/models/bluerov/urdf/bluerov_thrusters.xacro (robot description, xacro)
@@ -2,20 +2,20 @@
 <robot xmlns:xacro="http://www.ros.org/wiki/xacro">
   <!-- Adding the thruster units with the macro created in rov_example_snippets.xacro -->
-  <xacro:thruster_macro namespace="${namespace}" thruster_id="0">
+  <xacro:thruster_macro robot_namespace="${namespace}" thruster_id="0">
     <origin xyz="0.0 0.115 0.0" rpy="-0.0 -1.57079632679 0.0"/>
   </xacro:thruster_macro>
-  <xacro:thruster_macro namespace="${namespace}" thruster_id="1">
+  <xacro:thruster_macro robot_namespace="${namespace}" thruster_id="1">
     <origin xyz="0.0 -0.115 0.0" rpy="-0.0 -1.57079632679 0.0"/>
   </xacro:thruster_macro>
-  <xacro:thruster_macro namespace="${namespace}" thruster_id="2">
-    <origin xyz="0.18 0.1092 0.0" rpy="0.0 -0.0 0.0"//>
+  <xacro:thruster_macro robot_namespace="${namespace}" thruster_id="2">
+    <origin xyz="0.18 0.1092 0.0" rpy="0.0 -0.0 0.0"/>
   </xacro:thruster_macro>
-  <xacro:thruster_macro namespace="${namespace}" thruster_id="4">
+  <xacro:thruster_macro robot_namespace="${namespace}" thruster_id="4">
     <origin xyz="0.18 -0.1092 0.0" rpy="0.0 -0.0 0.0"/>
   </xacro:thruster_macro>
-  <xacro:thruster_macro namespace="${namespace}" thruster_id="5">
+  <xacro:thruster_macro robot_namespace="${namespace}" thruster_id="5">
     <origin  xyz="-0.17 0.0 0.0" rpy="0.0 -0.0 0.0"/>
   </xacro:thruster_macro>
-  <xacro:thruster_macro namespace="${namespace}" thruster_id="6">
+  <xacro:thruster_macro robot_namespace="${namespace}" thruster_id="6">
     <origin xyz="0.0 0.0 0.105" rpy="1.57079632679 -0.0 0.0"/>
   </xacro:thruster_macro>

Commit message: asdasdasd

File: bluerov_uuv/models/bluerov/urdf/bluerov_base.xacro (robot description, xacro)
@@ -125,7 +125,7 @@
     </gazebo>
     <!-- Include the thruster modules -->
-    <xacro:include filename="$(find bluerov_uuv)/models/bluerov/urdf/bluerov_thrusters.xacro"/>
+    <!-- <xacro:include filename="$(find bluerov_uuv)/models/bluerov/urdf/bluerov_thrusters.xacro"/> -->
     <!-- Include the sensor modules -->
-    <xacro:include filename="$(find bluerov_uuv)/models/bluerov/urdf/bluerov_sensors.xacro"/>
+    <!-- <xacro:include filename="$(find bluerov_uuv)/models/bluerov/urdf/bluerov_sensors.xacro"/> -->
   </xacro:macro>
 </robot>

File: enigma_description/urdf/actuators.xacro (robot description, xacro)
@@ -8,4 +8,16 @@
           aware that Gazebo does not use the SNAME convention per default.
     -->
+<!--    <xacro:macro name="thruster_macro"
+    params="namespace thruster_id *origin">
+    <xacro:thruster_module_first_order_basic_fcn_macro
+      namespace="${namespace}"
+      thruster_id="${thruster_id}"
+      dyn_time_constant="0.05"
+      mesh_filename=""
+      rotor_constant="0.00031">
+      <xacro:insert_block name="origin"/>
+    </xacro:thruster_module_first_order_basic_fcn_macro>
+  </xacro:macro>
+ -->
     <xacro:thruster_macro robot_namespace="${namespace}" thruster_id="0">
         <origin xyz="0.0 0.115 0.0" rpy="-0.0 -1.57079632679 0.0"/>

File: enigma_description/urdf/base.xacro (robot description, xacro)
@@ -7,4 +7,5 @@
   <!-- Loading vehicle's specific macros -->
   <xacro:include filename="$(find enigma_description)/urdf/snippets.xacro"/>
+  <!-- <xacro:include filename="$(find uuv_gazebo_ros_plugins)/urdf/snippets.xacro"/> -->
   <!--
     Vehicle's parameters (remember to enter the model parameters below)
@@ -21,5 +22,5 @@
     Open the meshes for the RexROV vehicle in Blender to see an example on the mesh placement.
   -->
-  <xacro:property name="visual_mesh_file" value="file://$(find enigma_description)/meshes/fixed_rov.dae"/>
+  <xacro:property name="visual_mesh_file" value="file://$(find enigma_description)/meshes/fix_rov.dae"/>
   <!-- <xacro:property name="visual_mesh_file" value="file://$(find enigma_description)/meshes/rex.dae"/> -->
   <!-- Collision geometry mesh, usually in STL format (it is recommended to keep
@@ -49,5 +50,5 @@
           <origin xyz="0 0 0" rpy="0 0 0"/>
           <geometry>
-            <mesh filename="${visual_mesh_file}" scale="0.1 0.1 0.1" />
+            <mesh filename="${visual_mesh_file}" scale="1 1 1" />
           </geometry>
         </collision>
@@ -59,5 +60,5 @@
     <xacro:insert_block name="gazebo"/>
     <!-- Include the thruster modules -->
-    <!-- <xacro:include filename="$(find enigma_description)/urdf/thrusters.xacro"/> -->
+    <!-- <xacro:include filename="$(find enigma_description)/urdf/actuators.xacro"/> -->
     <!-- Include the sensor modules -->
     <!-- <xacro:include filename="$(find enigma_description)/urdf/sensors.xacro"/> -->

File: enigma_description/urdf/gazebo.xacro (robot description, xacro)
@@ -6,7 +6,7 @@
     <xacro:property name="enigma_volume" value="1.83826"/>
     <!-- Describing the dimensions of the vehicle's bounding box -->
-    <xacro:property name="enigma_length" value="0"/>
+    <!-- <xacro:property name="enigma_length" value="0"/>
     <xacro:property name="enigma_width"  value="0"/>
-    <xacro:property name="enigma_height" value="0"/>
+    <xacro:property name="enigma_height" value="0"/> -->
     <xacro:property name="volume" value="1.83826"/>
     <xacro:macro name="enigma_hydro_model" params="namespace">

File: enigma_description/urdf/sensors.xacro (robot description, xacro)
@@ -7,23 +7,15 @@
     more examples or add you own custom sensor units.
   -->
-  <!-- Mount a GPS. -->
-  <xacro:default_gps namespace="${namespace}" parent_link="${namespace}/base_link" />
-  <!-- Mount a Pose 3D sensor. -->
-  <xacro:default_pose_3d namespace="${namespace}" parent_link="${namespace}/base_link" />
-  <!-- Forward-looking sonar sensor -->
-  <xacro:forward_multibeam_p900 namespace="${namespace}" parent_link="${namespace}/base_link">
-    <origin xyz="0 0 0" rpy="0 0 0"/>
-  </xacro:forward_multibeam_p900>
-  <!-- DVL  -->
+  <!-- Mount a DVL. -->
   <xacro:default_dvl namespace="${namespace}" parent_link="${namespace}/base_link">
-    <origin xyz="0 0 0" rpy="0 0 0"/>
+    <origin xyz="-1.4 0 -0.312" rpy="0 ${0.5*pi} 0"/>
   </xacro:default_dvl>
   <!-- RPT  -->
   <xacro:default_rpt namespace="${namespace}" parent_link="${namespace}/base_link">
-    <origin xyz="0 0 0" rpy="0 0 0"/>
+    <origin xyz="-1.32 0 0.8" rpy="0 0 0"/>
   </xacro:default_rpt>
   <!-- Pressure  -->
   <xacro:default_pressure namespace="${namespace}" parent_link="${namespace}/base_link">
-    <origin xyz="0 0 0" rpy="0 0 0"/>
+    <origin xyz="-1.15 0.25 0.6" rpy="0 0 0"/>
   </xacro:default_pressure>
   <!-- IMU  -->
@@ -32,6 +24,16 @@
   </xacro:default_imu>
   <!-- Mount a camera -->
-  <xacro:default_camera namespace="${namespace}" parent_link="${namespace}/base_link">
-    <origin xyz="0 0 0" rpy="0 0 0"/>
+  <xacro:default_camera namespace="${namespace}" parent_link="${namespace}/base_link" suffix="">
+    <origin xyz="1.15 0 0.4" rpy="0 0.6 0"/>
   </xacro:default_camera>
+  <xacro:default_camera namespace="${namespace}" parent_link="${namespace}/base_link" suffix="right">
+    <origin xyz="1.2 -0.8 0.8" rpy="0 0 0"/>
+  </xacro:default_camera>
+  <xacro:default_camera namespace="${namespace}" parent_link="${namespace}/base_link" suffix="left">
+    <origin xyz="1.2 0.9 0.8" rpy="0 0 0"/>
+  </xacro:default_camera>
+  <!-- Mount a GPS. -->
+  <xacro:default_gps namespace="${namespace}" parent_link="${namespace}/base_link" />
+  <!-- Mount a Pose 3D sensor. -->
+  <xacro:default_pose_3d namespace="${namespace}" parent_link="${namespace}/base_link" />
 </robot>

File: enigma_description/urdf/snippets.xacro (robot description, xacro)
@@ -1,16 +1,10 @@
 <?xml version="1.0"?>
 <robot xmlns:xacro="http://www.ros.org/wiki/xacro">
-  <!-------------------------------------------------------------------------->
-  <!-- MACRO FOR THRUSTER UNITS  -->
-  <!-------------------------------------------------------------------------->
   <!-- Provide the propeller mesh in a separate file with the rotation axis
   over propeller's frame X-axis in DAE (Collada) or STL format.
   -->
-  <!-- <xacro:property name="prop_mesh_file" value="file://$(find enigma_description)/meshes/propeller.dae"/> -->
-  <!--
-    Thruster macro with integration of joint and link. The thrusters should
-    be initialized in the actuators.xacro file.
-  -->
-  <!-- <xacro:macro name="thruster_macro" params="robot_namespace thruster_id *origin"> -->
+  <!-- <xacro:property name="prop_mesh_file" value="file://$(find uuv_descriptions_example)/models/rov_example/mesh/propeller.dae"/> -->
+  <!-- Thruster macro with integration of joint and link-->
+  <xacro:macro name="thruster_macro" params="robot_namespace thruster_id *origin">
     <!--
     Dummy link as place holder for the thruster frame,
@@ -18,10 +12,10 @@
     of the vehicle and may cause internal collisions if set otherwise
     -->
-    <!-- <link name="${robot_namespace}/thruster_${thruster_id}">
-      <visual>
+    <link name="${robot_namespace}/thruster_${thruster_id}">
+<!--       <visual>
         <geometry>
           <mesh filename="${prop_mesh_file}" scale="1 1 1" />
         </geometry>
-      </visual>
+      </visual> -->
       <inertial>
         <mass value="0.001" />
@@ -31,32 +25,116 @@
                izz="0.000000017" />
       </inertial>
-    </link> -->
+    </link>
     <!-- Joint between thruster link and vehicle base link -->
-    <!-- <joint name="${robot_namespace}/thruster_${thruster_id}_joint" type="continuous">
+    <joint name="${robot_namespace}/thruster_${thruster_id}_joint" type="continuous">
       <xacro:insert_block name="origin" />
       <axis xyz="1 0 0" />
       <parent link="${robot_namespace}/base_link" />
       <child link="${robot_namespace}/thruster_${thruster_id}" />
-    </joint> -->
-  <!-- <xacro:property name="prop_mesh_file" value="file://$(find uuv_descriptions)/models/rexrov/mesh/prop.dae"/> -->
-  <!-- Thruster joint and link snippet -->
-    <!-- <gazebo>
-      <plugin name="${namespace}_${thruster_id}_thruster_model" filename="libthruster_ros_plugin.so">
-        <linkName>${namespace}/thruster_${thruster_id}</linkName>
-        <jointName>${namespace}/thruster_${thruster_id}_joint</jointName>
-        <thrusterID>${thruster_id}</thrusterID>
+    </joint>
+    <gazebo>
+      <!-- Thruster ROS plugin -->
+      <plugin name="${robot_namespace}_${thruster_id}_thruster_model" filename="libthruster_ros_plugin.so">
+        <!-- Name of the thruster link -->
+        <linkName>${robot_namespace}/thruster_${thruster_id}</linkName>
+        <!-- Name of the joint between thruster and vehicle base link -->
+        <jointName>${robot_namespace}/thruster_${thruster_id}_joint</jointName>
+        <!-- Thruster force output topic name -->
+        <thrustTopic>${robot_namespace}/thrusters/${thruster_id}/thrust</thrustTopic>
+        <!-- Thruster commmand input topic name -->
+        <inputTopic>${robot_namespace}/thrusters/${thruster_id}/input</inputTopic>
+        <!-- Gain of the input command signal -->
+        <gain>1</gain>
+        <!-- Maximum allowed input value for the input signal for thruster unit -->
+        <clampMax>0</clampMax>
+        <!-- Minimum allowed value for the input signal for thruster unit -->
+        <clampMin>0</clampMin>
+        <!--
+        Value from 0 to 1 to set the efficiency of the output thrust force
+        Default value is 1.0
+        -->
+        <thrust_efficiency>1</thrust_efficiency>
+        <!--
+        Value from 0 to 1 to set the efficiency of the propeller as a factor
+        to be multiplied to the current value of the state variable at each
+        iteration.
+        Default value is 1.0
+        -->
+        <propeller_efficiency>1</propeller_efficiency>
+        <!-- Simple zero-order model -->
+        <dynamics>
+          <type>ZeroOrder</type>
+        </dynamics>
+        <!-- First order model, gain used is specified above -->
         <dynamics>
           <type>FirstOrder</type>
-          <timeConstant>0.05</timeConstant>urdf
+          <timeConstant>0.0</timeConstant>
         </dynamics>
+        <!-- Yoerger's nonlinear dynamic model
+        For information on the model description:
+        D. R. Yoerger, J. G. Cooke, and J.-J. E. Slotine, “The influence of
+        thruster dynamics on underwater vehicle behavior and their incorporation
+        into control system design,” IEEE Journal of Oceanic Engineering, vol. 15, no. 3, pp. 167–178, Jul. 1990.
+        -->
+        <dynamics>
+          <type>Yoerger</type>
+          <alpha>0.0</alpha>
+          <beta>0.0</beta>
+        </dynamics>
+        <!-- Bessa's nonlinear dynamic model
+        For information on the model description:
+        Bessa, Wallace Moreira, Max Suell Dutra, and Edwin Kreuzer. "Thruster
+        dynamics compensation for the positioning of underwater robotic vehicles
+        through a fuzzy sliding mode based approach." ABCM Symposium Series in
+        Mechatronics. Vol. 2. 2006.
+        -->
+        <dynamics>
+          <type>Bessa</type>
+          <Jmsp>0.0</Jmsp>
+          <Kv1>0.0</Kv1>
+          <Kv2>0.0</Kv2>
+          <Kt>0.0</Kt>
+          <Rm>0.0</Rm>
+        </dynamics>
+        <!-- Basic curve
+        Input: x
+        Output: thrust
+        Function: thrust = rotorConstant * x * abs(x)
+        -->
         <conversion>
           <type>Basic</type>
-          <rotorConstant>0.00031</rotorConstant>
+          <rotorConstant>0.0</rotorConstant>
+        </conversion>
+        <!-- Dead-zone nonlinearity described in Bessa, 2006
+        Input: x
+        Output: thrust
+        Function:
+        thrust = rotorConstantL * (x * abs(x) - deltaL), if x * abs(x) <= deltaL
+        thrust = 0, if deltaL < x * abs(x) < deltaR
+        thrust = rotorConstantR * (x * abs(x) - deltaR), if x * abs(x) >= deltaL
+        -->
+        <conversion>
+          <type>Bessa</type>
+          <rotorConstantL>0.0</rotorConstantL>
+          <rotorConstantR>0.0</rotorConstantR>
+          <deltaL>0.0</deltaL>
+          <deltaR>0.0</deltaR>
+        </conversion>
+        <!-- Linear interpolation
+        If you have access to the thruster's data sheet, for example,
+        you can enter samples of the curve's input and output values
+        and the thruster output will be found through linear interpolation
+        of the given samples.
+        -->
+        <conversion>
+          <type>LinearInterp</type>
+          <inputValues>0 1 2 3</inputValues>
+          <outputValues>0 1 2 3</outputValues>
         </conversion>
       </plugin>
     </gazebo>
-    <gazebo reference="${robot_namespace}/thruster_${thruster_id}">
+<!--     <gazebo reference="${robot_namespace}/thruster_${thruster_id}">
       <selfCollide>false</selfCollide>
-    </gazebo>
-  </xacro:macro> -->
+    </gazebo> -->
+  </xacro:macro>
 </robot>
